Commit message: -_-

File: hexapod_ws/src/hexapodV2/urdf/hexapodV2.urdf (robot description, URDF)
Before this commit: robot hexapodV2, 25 links, 24 joints
Joints:
- joint rb_toe: limit lower=-2.0944 upper=1.4835 effort=0.79796 velocity=5.235 -> lower=-1.4835 upper=2.0944 effort=0.79796 velocity=5.235
- joint rf_toe: limit lower=-2.0944 upper=1.4835 effort=0.79796 velocity=5.235 -> lower=-1.4835 upper=2.0994 effort=0.79796 velocity=5.235
- joint rm_toe: limit lower=-2.0944 upper=1.4835 effort=0.79796 velocity=5.235 -> lower=-1.4835 upper=2.0994 effort=0.79796 velocity=5.235
