Commit message: Control is better but not good, inertias bad

File: test_ws/src/hexapodV2/urdf/hexapodV2.urdf (robot description, URDF)
Before this commit: robot hexapodV2, 25 links, 24 joints
Links:
- added link base
Joints:
- added joint base_to_base_link: type fixed, parent base, child base_link, origin xyz=0 0 0 rpy=0 0 0
